File: power_p3v3.kicad_pcb (KiCad board)
At the start: 4 copper layers, 44.8 x 41.5 mm, 24 parts, among them J1 LSHM-140-04.0-L-DV-A-N-K-TR, U1 LT8627SP

Commit message: Add Ferrite Beads
Parts:
- added C12: 100u, lib:T521X, F.Cu at (126.4, 53.5)
- added R6: 0.5, Resistor_SMD:R_0603_1608Metric, F.Cu at (121.3, 52.5)
Routing:
- net /cf1: track 0.00 -> 4.97 mm
- net /PG: track 29.1 -> 27.9 mm
- net /SYNC: track 26.8 -> 25.7 mm
- net GND: vias 168 -> 165
